File: PCB/totemball_PCB/totem_0_3.kicad_pcb (KiCad board)
At the start: 2 copper layers, 238.6 x 94.4 mm, 96 parts, among them J3 Conn_01x06_MountingPin, J4 Conn_01x06_MountingPin, U1 xiao-ble, U2 xiao-ble

Commit message: fix errors
Routing:
- net COL4_L: track 183.3 -> 175.0 mm
- net RESET_R: track 104.0 -> 98.2 mm
- net ROW3_L: track 203.6 -> 200.6 mm
- net COL2_R: track 136.7 -> 135.0 mm
- net COL3_L: track 143.3 -> 141.9 mm
- net COL2_L: track 122.9 -> 121.5 mm
- net COL3_R: track 160.2 -> 159.0 mm
- net BAT+_R: track 29.5 -> 28.7 mm
- net RESET_L: track 116.0 -> 115.2 mm
- net COL1_R: track 64.8 -> 64.0 mm
- net CS_R: track 163.0 -> 163.6 mm
- net Motion_R: track 173.0 -> 172.5 mm
- net GND_L: vias 30 -> 27
Other:
- board text removed: "0.1"
- board text removed: "RX"
