File: PCB/totemball_PCB/totem_0_3.kicad_pcb (KiCad board)
At the start: 2 copper layers, 238.6 x 94.4 mm, 96 parts, among them J3 Conn_01x06_MountingPin, J4 Conn_01x06_MountingPin, U1 xiao-ble, U2 xiao-ble

Commit message: move ffc connector
Parts:
- moved J4 2.05 mm to (159.6, 104.4)
- moved J3 1.81 mm to (140.4, 104.1)
Routing:
- net SDIO_R: track 164.2 -> 166.2 mm
- net Motion_R: track 172.5 -> 174.6 mm
- net VCC_R: track 169.9 -> 171.9 mm
- net SLCK_R: track 167.8 -> 169.9 mm
- net CS_R: track 163.6 -> 165.6 mm
- net SDIO_L: track 176.6 -> 178.4 mm
- net SLCK_L: track 160.2 -> 162.0 mm
- net Motion_L: track 177.3 -> 179.0 mm
- net VCC_L: track 177.6 -> 179.2 mm
- net CS_L: track 159.4 -> 161.0 mm
