File: PCB/totemball_PCB/totem_0_3.kicad_pcb (KiCad board)
At the start: 2 copper layers, 238.6 x 94.4 mm, 96 parts, among them J3 Conn_01x06_MountingPin, J4 Conn_01x06_MountingPin, U1 xiao-ble, U2 xiao-ble

Commit message: add pochita
Parts:
- added G*** (x2): LOGO, LOGO, B.Cu at (226.8, 112.0)
- added G*** (x2): LOGO, LOGO, B.Cu at (89.2, 107.2)
- added G*** (x2): LOGO, LOGO, B.Cu at (74.0, 110.2)
Routing:
- net COL2_L: track 121.5 -> 126.5 mm
